File: hardware/tick-display-mk-3-mini.sch (EAGLE design)
At the start: 18 parts, among them IC1 ATTINY84, IC2 DS1307, IC3 74595DIP, Y1 32.768kHz

Commit message: scaled down even more
Parts:
- removed TEMP_C: 7SEG_2DIG, A_butts:7SEG_2DIG
- added AVRISP: AVR_SPI_PRG_6PTH, A_butts:AVR_SPI_PRG_6PTH
- added BATT: M02JST-PTH-VERT, A_butts:M02JST-PTH-VERT
- added C4: 10uF, A_butts:CAPACITOR-POLARIZEDE2.5-6
- added C5: 100uF, A_butts:CAPACITOR-POLARIZEDE2.5-6
- added D1: 1N5819, A_butts:DIODE-SCHOTTKYPTH-10.16MM
- added DC_IN: (no value), A_butts:DCBARRELPTH
- added F1: PTCPTH, A_butts:PTCPTH
- added IC4: LM2931, A_butts:V_REG_78XXTO-92-INLINE
- added LED1: LED3MM, A_butts:LED3MM
- added R6: 330R, A_butts:RESISTORPTH-AXIAL-5.08MM
- added RST: SPST-NO-TACT3MM-PTH-SMALL-PADS, A_butts:SPST-NO-TACT3MM-PTH-SMALL-PADS
- added TVS1: (no value), A_butts:TVSDO-41-TVS-BIDIRECTIONAL
- IC3: value 74595DIP -> 74HCT595
- renumbered TIME to DISPLAY
Connections:
- removed net TC1: IC1.(PCINT1/AIN0/ADC1)PA1, TEMP_C.DIG1
- removed net TC2: IC1.(PCINT0/AREF/ADC0)PA0, TEMP_C.DIG2
- new net DP: DISPLAY.DP, IC3.QH
- new net MISO: AVRISP.MISO, IC1.(PCINT5/OC1B/MISO/DO/ADC5)PA5
- new net N$1: BATT.1, IC2.VBAT
- new net N$10: LED1.A, R6.2
- new net N$3: DC_IN.PWR, F1.1
- new net N$5: C4.+, D1.C, IC4.IN
- new net RESET: AVRISP.RESET, IC1.(PCINT11/~RESET/DW)PB3, R1.1, RST.1
- net A: no longer TEMP_C.A
- net B: no longer TEMP_C.B
- net C: no longer TEMP_C.C
- net D: no longer TEMP_C.D
- net E: no longer TEMP_C.E
- net F: no longer TEMP_C.F
- net G: no longer TEMP_C.G
- net GND: now also AVRISP.GND, BATT.2, C4.-, C5.-, DC_IN.BRK, DC_IN.GND, IC4.GND, LED1.C, RST.2, TVS1.1
- net HR1: now also IC1.(PCINT3/T0/ADC3)PA3; no longer IC1.(PCINT7/ICP/OC0B/ADC7)PA7
- net HR2: now also IC1.(PCINT2/AIN1/ADC2)PA2; no longer IC1.(PCINT5/OC1B/MISO/DO/ADC5)PA5
- net MI1: now also IC1.(PCINT1/AIN0/ADC1)PA1; no longer IC1.(PCINT3/T0/ADC3)PA3
- net MI2: now also IC1.(PCINT0/AREF/ADC0)PA0; no longer IC1.(PCINT2/AIN1/ADC2)PA2
- net N$4: now also D1.A, F1.2, TVS1.2; no longer IC1.(PCINT11/~RESET/DW)PB3, R1.1
- net SCL: now also AVRISP.SCK
- net SDA: now also AVRISP.MOSI
- net VCC: now also AVRISP.VCC, C5.+, IC4.OUT, R6.1
Other:
- moved on the sheet: IC2, Y1

Commit message: again with the not sure what the fuck i was thinking
Parts:
- removed H1, H2, H3, H4: HOLE#2, A_butts:HOLE#2
- D1: device A_butts:DIODE-SCHOTTKYPTH-10.16MM -> A_butts:DIODE-SCHOTTKYPTH-7.68MM
- DISPLAY: value 7SED_4DIGIT_14MM14.2MM-CC -> 7SED_4DIGIT_14MM14.2MM-CC-NS; device A_butts:7SED_4DIGIT_14MM14.2MM-CC -> A_butts:7SED_4DIGIT_14MM14.2MM-CC-NS
- RST: value SPST-NO-TACT3MM-PTH-SMALL-PADS -> SPST-NO-TACT3MM-RA; device A_butts:SPST-NO-TACT3MM-PTH-SMALL-PADS -> A_butts:SPST-NO-TACT3MM-RA
Connections:
- net B: now also IC3.QH; no longer IC3.QB
- net C: now also IC3.QE; no longer IC3.QC
- net D: now also IC3.QC; no longer IC3.QD
- net DP: now also IC3.QD; no longer IC3.QH
- net E: now also IC3.QB; no longer IC3.QE
- net F: now also IC3.QG; no longer IC3.QF
- net G: now also IC3.QF; no longer IC3.QG
Changed lines of the file:
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@@
 </classes>
 <parts>
-<part name="DISPLAY" library="A_butts" deviceset="7SED_4DIGIT_14MM" device="14.2MM-CC"/>
+<part name="DISPLAY" library="A_butts" deviceset="7SED_4DIGIT_14MM" device="14.2MM-CC-NS" value="7SED_4DIGIT_14MM14.2MM-CC-NS"/>
 <part name="SUPPLY5" library="A_butts" deviceset="VCC" device=""/>
 <part name="SUPPLY8" library="A_butts" deviceset="VCC" device=""/>
@@
 <part name="SUPPLY2" library="A_butts" deviceset="VCC" device=""/>
 <part name="GND2" library="A_butts" deviceset="GND" device=""/>
-<part name="H3" library="A_butts" deviceset="HOLE" device="#2" value="HOLE#2"/>
-<part name="H4" library="A_butts" deviceset="HOLE" device="#2" value="HOLE#2"/>
 <part name="R3" library="A_butts" deviceset="RESISTOR" device="PTH-AXIAL-5.08MM" value="330R"/>
 <part name="IC2" library="A_butts" deviceset="DS1307" device=""/>
@@
 <part name="SUPPLY10" library="A_butts" deviceset="VCC" device=""/>
 <part name="Y1" library="A_butts" deviceset="CRYSTAL" device="TC26H" value="32.768kHz"/>
-<part name="H1" library="A_butts" deviceset="HOLE" device="#2" value="HOLE#2"/>
-<part name="H2" library="A_butts" deviceset="HOLE" device="#2" value="HOLE#2"/>
 <part name="IC1" library="A_butts" deviceset="ATTINY84" device="ATTINY84-20PU" value="ATTINY84"/>
 <part name="IC3" library="A_butts" deviceset="74*595" device="DIP" value="74HCT595"/>
@@
 <part name="IC4" library="A_butts" deviceset="V_REG_78XX" device="TO-92-INLINE" value="LM2931"/>
 <part name="F1" library="A_butts" deviceset="PTC" device="PTH"/>
-<part name="D1" library="A_butts" deviceset="DIODE-SCHOTTKY" device="PTH-10.16MM" value="1N5819"/>
+<part name="D1" library="A_butts" deviceset="DIODE-SCHOTTKY" device="PTH-7.68MM" value="1N5819"/>
 <part name="C4" library="A_butts" deviceset="CAPACITOR-POLARIZED" device="E2.5-6" value="10uF"/>
 <part name="C5" library="A_butts" deviceset="CAPACITOR-POLARIZED" device="E2.5-6" value="100uF"/>
 <part name="TVS1" library="A_butts" deviceset="TVS" device="DO-41-TVS-BIDIRECTIONAL"/>
-<part name="RST" library="A_butts" deviceset="SPST-NO-TACT" device="3MM-PTH-SMALL-PADS" value="SPST-NO-TACT3MM-PTH-SMALL-PADS"/>
+<part name="RST" library="A_butts" deviceset="SPST-NO-TACT" device="3MM-RA" value="SPST-NO-TACT3MM-RA"/>
 <part name="AVRISP" library="A_butts" deviceset="AVR_SPI_PRG_6" device="PTH"/>
 <part name="GND3" library="A_butts" deviceset="GND" device=""/>
@@
 <instance part="SUPPLY2" gate="G$1" x="30.48" y="172.72"/>
 <instance part="GND2" gate="1" x="30.48" y="154.94"/>
-<instance part="H3" gate="G$1" x="15.24" y="187.96"/>
-<instance part="H4" gate="G$1" x="20.32" y="187.96"/>
 <instance part="R3" gate="G$1" x="71.12" y="58.42"/>
 <instance part="IC2" gate="G$1" x="-5.08" y="119.38"/>
@@
 <instance part="SUPPLY10" gate="G$1" x="12.7" y="172.72"/>
 <instance part="Y1" gate="G$1" x="-7.62" y="142.24" rot="MR0"/>
-<instance part="H1" gate="G$1" x="5.08" y="187.96"/>
-<instance part="H2" gate="G$1" x="10.16" y="187.96"/>
 <instance part="IC1" gate="G$1" x="53.34" y="116.84"/>
 <instance part="IC3" gate="G$1" x="127" y="76.2"/>
@@
 </segment>
 <segment>
+<pinref part="IC3" gate="G$1" pin="QH"/>
+<wire x1="142.24" y1="68.58" x2="144.78" y2="68.58" width="0.1524" layer="91"/>
+<label x="144.78" y="68.58" size="1.27" layer="95" xref="yes"/>
+</segment>
+</net>
+<net name="D" class="0">
+<segment>
+<pinref part="DISPLAY" gate="G$1" pin="D"/>
+<wire x1="15.24" y1="66.04" x2="17.78" y2="66.04" width="0.1524" layer="91"/>
+<label x="15.24" y="66.04" size="1.27" layer="95" rot="R180" xref="yes"/>
+</segment>
+<segment>
+<wire x1="144.78" y1="81.28" x2="142.24" y2="81.28" width="0.1524" layer="91"/>
+<label x="144.78" y="81.28" size="1.27" layer="95" xref="yes"/>
+<pinref part="IC3" gate="G$1" pin="QC"/>
+</segment>
+</net>
+<net name="F" class="0">
+<segment>
+<pinref part="DISPLAY" gate="G$1" pin="F"/>
+<wire x1="15.24" y1="60.96" x2="17.78" y2="60.96" width="0.1524" layer="91"/>
+<label x="15.24" y="60.96" size="1.27" layer="95" rot="R180" xref="yes"/>
+</segment>
+<segment>
+<wire x1="144.78" y1="71.12" x2="142.24" y2="71.12" width="0.1524" layer="91"/>
+<label x="144.78" y="71.12" size="1.27" layer="95" xref="yes"/>
+<pinref part="IC3" gate="G$1" pin="QG"/>
+</segment>
+</net>
+<net name="G" class="0">
+<segment>
+<pinref part="DISPLAY" gate="G$1" pin="G"/>
+<wire x1="15.24" y1="58.42" x2="17.78" y2="58.42" width="0.1524" layer="91"/>
+<label x="15.24" y="58.42" size="1.27" layer="95" rot="R180" xref="yes"/>
+</segment>
+<segment>
+<wire x1="144.78" y1="73.66" x2="142.24" y2="73.66" width="0.1524" layer="91"/>
+<label x="144.78" y="73.66" size="1.27" layer="95" xref="yes"/>
+<pinref part="IC3" gate="G$1" pin="QF"/>
+</segment>
+</net>
+<net name="E" class="0">
+<segment>
+<pinref part="DISPLAY" gate="G$1" pin="E"/>
+<wire x1="15.24" y1="63.5" x2="17.78" y2="63.5" width="0.1524" layer="91"/>
+<label x="15.24" y="63.5" size="1.27" layer="95" rot="R180" xref="yes"/>
+</segment>
+<segment>
 <wire x1="144.78" y1="83.82" x2="142.24" y2="83.82" width="0.1524" layer="91"/>
 <label x="144.78" y="83.82" size="1.27" layer="95" xref="yes"/>
@@
 </segment>
 </net>
-<net name="D" class="0">
-<segment>
-<pinref part="DISPLAY" gate="G$1" pin="D"/>
-<wire x1="15.24" y1="66.04" x2="17.78" y2="66.04" width="0.1524" layer="91"/>
-<label x="15.24" y="66.04" size="1.27" layer="95" rot="R180" xref="yes"/>
-</segment>
-<segment>
-<wire x1="144.78" y1="78.74" x2="142.24" y2="78.74" width="0.1524" layer="91"/>
-<label x="144.78" y="78.74" size="1.27" layer="95" xref="yes"/>
-<pinref part="IC3" gate="G$1" pin="QD"/>
-</segment>
-</net>
-<net name="F" class="0">
-<segment>
-<pinref part="DISPLAY" gate="G$1" pin="F"/>
-<wire x1="15.24" y1="60.96" x2="17.78" y2="60.96" width="0.1524" layer="91"/>
-<label x="15.24" y="60.96" size="1.27" layer="95" rot="R180" xref="yes"/>
-</segment>
-<segment>
-<wire x1="144.78" y1="73.66" x2="142.24" y2="73.66" width="0.1524" layer="91"/>
-<label x="144.78" y="73.66" size="1.27" layer="95" xref="yes"/>
-<pinref part="IC3" gate="G$1" pin="QF"/>
-</segment>
-</net>
-<net name="G" class="0">
-<segment>
-<pinref part="DISPLAY" gate="G$1" pin="G"/>
-<wire x1="15.24" y1="58.42" x2="17.78" y2="58.42" width="0.1524" layer="91"/>
-<label x="15.24" y="58.42" size="1.27" layer="95" rot="R180" xref="yes"/>
-</segment>
-<segment>
-<wire x1="144.78" y1="71.12" x2="142.24" y2="71.12" width="0.1524" layer="91"/>
-<label x="144.78" y="71.12" size="1.27" layer="95" xref="yes"/>
-<pinref part="IC3" gate="G$1" pin="QG"/>
-</segment>
-</net>
-<net name="E" class="0">
-<segment>
-<pinref part="DISPLAY" gate="G$1" pin="E"/>
-<wire x1="15.24" y1="63.5" x2="17.78" y2="63.5" width="0.1524" layer="91"/>
-<label x="15.24" y="63.5" size="1.27" layer="95" rot="R180" xref="yes"/>
+<net name="C" class="0">
+<segment>
+<pinref part="DISPLAY" gate="G$1" pin="C"/>
+<wire x1="15.24" y1="68.58" x2="17.78" y2="68.58" width="0.1524" layer="91"/>
+<label x="15.24" y="68.58" size="1.27" layer="95" rot="R180" xref="yes"/>
 </segment>
 <segment>
@@
 <label x="144.78" y="76.2" size="1.27" layer="95" xref="yes"/>
 <pinref part="IC3" gate="G$1" pin="QE"/>
-</segment>
-</net>
-<net name="C" class="0">
-<segment>
-<pinref part="DISPLAY" gate="G$1" pin="C"/>
-<wire x1="15.24" y1="68.58" x2="17.78" y2="68.58" width="0.1524" layer="91"/>
-<label x="15.24" y="68.58" size="1.27" layer="95" rot="R180" xref="yes"/>
-</segment>
-<segment>
-<wire x1="144.78" y1="81.28" x2="142.24" y2="81.28" width="0.1524" layer="91"/>
-<label x="144.78" y="81.28" size="1.27" layer="95" xref="yes"/>
-<pinref part="IC3" gate="G$1" pin="QC"/>
 </segment>
 </net>
@@
 </segment>
 <segment>
-<pinref part="IC3" gate="G$1" pin="QH"/>
-<wire x1="142.24" y1="68.58" x2="144.78" y2="68.58" width="0.1524" layer="91"/>
-<label x="144.78" y="68.58" size="1.27" layer="95" xref="yes"/>
+<wire x1="144.78" y1="78.74" x2="142.24" y2="78.74" width="0.1524" layer="91"/>
+<label x="144.78" y="78.74" size="1.27" layer="95" xref="yes"/>
+<pinref part="IC3" gate="G$1" pin="QD"/>
 </segment>
 </net>
@@
 </sheet>
 </sheets>
+<errors>
+</errors>
 </schematic>
 </drawing>
