File: hardware/tick-shield-mk-1.sch (EAGLE design)
At the start: 15 parts, among them IC1 DS1307, Y1 32.768kHz

Commit message: shieldify all the things
Parts:
- removed C3: 1uF, A_butts:CAPACITOR-CERAMICC0805
- removed DISPLAY3, DISPLAY4: 7SEG_4DIGIT_COLON_APOS, A_butts:7SEG_4DIGIT_COLON_APOS
- removed Y1: 32.768kHz, A_butts:CRYSTALTC26H
- added R1, R2: 4.7k, A_butts:RESISTORR0603
- C2: value 0.1uF -> 1uF; device A_butts:CAPACITOR-CERAMICC0603 -> A_butts:CAPACITOR-CERAMICC0805
- DISPLAY2: value 7SEG_4DIGIT_COLON_APOS -> 7SEG_4DIGIT_COLON14.2MM-CC; device A_butts:7SEG_4DIGIT_COLON_APOS -> A_butts:7SEG_4DIGIT_COLON14.2MM-CC
- IC1: value DS1307 -> DS1338C; device A_butts:DS1307 -> A_butts:DS1338CSOIC16W
Connections:
- removed net D10: DISPLAY1.A, DISPLAY2.A, DISPLAY3.DIG1, SHIELD.*D10
- removed net D11: DISPLAY1.B, DISPLAY2.B, DISPLAY3.DIG2, SHIELD.*D11
- removed net D12: DISPLAY1.C, DISPLAY2.C, DISPLAY3.DIG3, SHIELD.D12
- removed net D13: DISPLAY1.D, DISPLAY2.D, DISPLAY3.DIG4, SHIELD.D13
- removed net N$1: IC1.X2, Y1.2
- removed net N$2: IC1.X1, Y1.1
- net A0: now also DISPLAY1.A; no longer DISPLAY1.E, DISPLAY4.DIG1
- net A1: now also DISPLAY1.B; no longer DISPLAY1.F, DISPLAY4.DIG2
- net A2: now also DISPLAY1.C; no longer DISPLAY1.G, DISPLAY4.DIG3
- net A3: now also DISPLAY1.D; no longer DISPLAY1.DP, DISPLAY4.DIG4
- net D2: now also DISPLAY1.E, DISPLAY2.DIG1; no longer DISPLAY1.DIG1, DISPLAY3.A, DISPLAY4.A
- net D3: now also DISPLAY1.F, DISPLAY2.DIG2; no longer DISPLAY1.DIG2, DISPLAY3.B, DISPLAY4.B
- net D4: now also DISPLAY1.G, DISPLAY2.DIG3; no longer DISPLAY1.DIG3, DISPLAY3.C, DISPLAY4.C
- net D5: now also DISPLAY1.DP, DISPLAY2.DIG4; no longer DISPLAY1.DIG4, DISPLAY3.D, DISPLAY4.D
- net D6: now also DISPLAY1.DIG1, DISPLAY2.A; no longer DISPLAY2.DIG1, DISPLAY3.E, DISPLAY4.E
- net D7: now also DISPLAY1.DIG2, DISPLAY2.B; no longer DISPLAY2.DIG2, DISPLAY3.F, DISPLAY4.F
- net D8: now also DISPLAY1.DIG3, DISPLAY2.C; no longer DISPLAY2.DIG3, DISPLAY3.G, DISPLAY4.G
- net D9: now also DISPLAY1.DIG4, DISPLAY2.D; no longer DISPLAY2.DIG4, DISPLAY3.DP, DISPLAY4.DP
- net GND: no longer C3.2
- net N$3: now also IC1.VBATT; no longer IC1.VBAT
- net SCL: now also R2.1
- net SDA: now also R1.1
- net VCC: now also R1.2, R2.2; no longer C3.1
Other:
- moved on the sheet: BAT1
