File: hardware/tick-mk-4.1.brd (EAGLE design)
At the start: 96 x 53 mm, 15 parts, among them U1 ATMEGA328P

Commit message: routed and RTC chip added
Parts:
- added AVR_ISP: AVR_SPI_PRG_6PTH, A_butts:2X3
- added C3: 0.1uF, A_butts:C0805
- added C4: 1uF, A_butts:C0805
- added IC2: DS1338, A_butts:SO16W
- added R2, R3: 4.7k, A_butts:R0805
- C1: value 1uF -> 0.1uF
- Y1: value (none) -> 16MHz
- renumbered U1 to IC1
Connections:
- new net D10: DISPLAY1.3, DISPLAY2.8, IC1.14
- new net D11/MOSI: AVR_ISP.4, IC1.15
- new net D12/MISO: AVR_ISP.1, IC1.16
- new net D13/SCK: AVR_ISP.3, IC1.17
- net A0: now also DISPLAY1.5, DISPLAY2.14
- net A1: now also DISPLAY1.11, DISPLAY2.16
- net A2: now also DISPLAY1.15, DISPLAY2.13
- net A3: now also DISPLAY1.7, DISPLAY2.3
- net D0: now also DISPLAY2.5
- net D1: now also DISPLAY2.11
- net D2: now also DISPLAY2.15
- net D3: now also DISPLAY1.1, DISPLAY2.7
- net D4: now also DISPLAY1.2
- net D5: now also DISPLAY1.6
- net D6: now also DISPLAY1.8
- net D7: now also DISPLAY1.14, DISPLAY2.1
- net D8: now also DISPLAY1.16, DISPLAY2.2
- net D9: now also DISPLAY1.13, DISPLAY2.6
- net GND: now also AVR_ISP.6, C3.2, C4.2, IC2.10, IC2.11, IC2.12, IC2.13, IC2.15, IC2.4, IC2.5, IC2.6, IC2.7, IC2.8, IC2.9
- net RST: now also AVR_ISP.5
- net SCL: now also IC2.1, R3.2
- net SDA: now also IC2.16, R2.2
- net VCC: now also AVR_ISP.2, C3.1, C4.1, IC2.3, R2.1, R3.1
Routing:
- net D3: track 94.3 -> 185.4 mm, vias 5 -> 9
- net D10: track 0.00 -> 78.6 mm, vias 0 -> 4
- net A0: track 117.6 -> 181.7 mm, vias 3 -> 7
- net D9: track 0.00 -> 63.3 mm, vias 0 -> 3
- net D8: track 0.00 -> 59.5 mm, vias 0 -> 2
- net VCC: track 17.9 -> 74.3 mm, vias 0 -> 3
- net D7: track 0.00 -> 52.6 mm, vias 0 -> 2
- net A1: track 107.3 -> 156.6 mm, vias 3 -> 5
- net SCL: track 0.00 -> 43.9 mm, vias 0 -> 2
- net SDA: track 0.00 -> 37.3 mm, vias 0 -> 2
- net A3: track 89.8 -> 127.0 mm, vias 5 -> 6
- net D2: track 94.9 -> 129.6 mm, vias 4 -> 7
- net D5: track 0.00 -> 31.0 mm, vias 0 -> 2
- net RST: track 3.63 -> 30.3 mm, vias 0 -> 1
- net D11/MOSI: track 0.00 -> 26.1 mm
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