File: hardware/tick-mk-4.7.brd (EAGLE design)
At the start: 96 x 54 mm, 39 parts, among them IC1 TINY85-20-DIP, IC2 DS1307, IC3 L7805, IC4 MAX7219, IC5 MAX7219, J1 PROG, Y2 32.768kHz

Commit message: diddling
Parts:
- added C6: 10uF, A_butts:E2-5
- added C7: 100uF, A_butts:E2,5-6
- C3: value 1uF -> 0.1uF
- C4: value 10uF -> 0.1uF; device A_butts:E2-5 -> A_butts:C025-024X044
- C5: value 100uF -> 1uF; device A_butts:E2,5-6 -> A_butts:C025-024X044
- moved C4 88.9 mm to (-3.00, -4.50)
- moved C5 82.3 mm to (-3.00, -7.00), turned to 0 degrees
- moved R5 46.1 mm to (50.9, 62.3)
- moved C1 45.9 mm to (73.2, 61.0)
- moved R4 43.3 mm to (62.9, 61.9)
- moved IC4 25.0 mm to (48.0, 7.10), turned to 0 degrees
- moved IC5 12.2 mm to (48.2, 27.0)
Connections:
- net N$15 renamed DIG15
- net N$16 renamed DIG14
- net N$17 renamed DIG13
- net N$18 renamed DIG12
- removed net N$10: IC4.13
- removed net N$13: IC5.12
- removed net N$14: IC5.13
- removed net N$19: IC5.7
- removed net N$20: IC5.6
- removed net N$21: IC5.11
- removed net N$22: IC5.2
- removed net N$23: IC4.8
- removed net N$24: IC4.5
- removed net N$25: IC4.10
- removed net N$26: IC4.3
- removed net N$27: IC4.7
- removed net N$28: IC4.6
- removed net N$29: IC4.11
- removed net N$30: IC4.2
- removed net N$31: IC4.1
- removed net N$32: IC5.17
- removed net N$9: IC4.12
- new net A1: DISPLAY1.14, DISPLAY2.14, IC4.14
- new net A2: DIGIT1.7, DIGIT2.7, DIGIT3.7, DIGIT4.7, IC5.14
- new net B1: DISPLAY1.16, DISPLAY2.16, IC4.16
- new net B2: DIGIT1.6, DIGIT2.6, DIGIT3.6, DIGIT4.6, IC5.16
- new net C1: DISPLAY1.13, DISPLAY2.13, IC4.20
- new net C2: DIGIT1.4, DIGIT2.4, DIGIT3.4, DIGIT4.4, IC5.20
- new net D1: DISPLAY1.3, DISPLAY2.3, IC4.23
- new net D2: DIGIT1.2, DIGIT2.2, DIGIT3.2, DIGIT4.2, IC5.23
- new net DIG0: DISPLAY1.1, IC4.2
- new net DIG1: DISPLAY1.2, IC4.11
- new net DIG10: DIGIT3.3, DIGIT3.8, IC5.6
- new net DIG11: DIGIT4.3, DIGIT4.8, IC5.7
- new net DIG2: DISPLAY1.6, IC4.6
- new net DIG3: DISPLAY1.8, IC4.7
- new net DIG4: DISPLAY2.1, IC4.3
- new net DIG5: DISPLAY2.2, IC4.10
- new net DIG6: DISPLAY2.6, IC4.5
- new net DIG7: DISPLAY2.8, IC4.8
- new net DIG8: DIGIT1.3, DIGIT1.8, IC5.2
- new net DIG9: DIGIT2.3, DIGIT2.8, IC5.11
- new net DP1: DISPLAY1.7, DISPLAY2.7, IC4.22
- new net DP2: DIGIT1.5, DIGIT2.5, DIGIT3.5, DIGIT4.5, IC5.22
- new net E1: DISPLAY1.5, DISPLAY2.5, IC4.21
- new net E2: DIGIT1.1, DIGIT2.1, DIGIT3.1, DIGIT4.1, IC5.21
- new net F1: DISPLAY1.11, DISPLAY2.11, IC4.15
- new net F2: DIGIT1.9, DIGIT2.9, DIGIT3.9, DIGIT4.9, IC5.15
- new net G1: DISPLAY1.15, DISPLAY2.15, IC4.17
- new net G2: DIGIT1.10, DIGIT2.10, DIGIT3.10, DIGIT4.10, IC5.17
- net CLK: now also IC4.13, IC5.13
- net DIN: now also IC4.1
- net GND: now also C4.2, C5.2, C6.-, C7.-, IC4.4, IC4.9, IC5.4, IC5.9; no longer C4.-, C5.-
- net LOAD: now also IC4.12, IC5.12
- net N$8: now also C6.+; no longer C4.+
- net VCC: now also C4.1, C5.1, C7.+; no longer C5.+

Commit message: commit before pull
Parts:
- moved R4 104.9 mm to (0.00, -22.0)
- moved IC5 61.4 mm to (3.00, -14.5), turned to 0 degrees
- moved C2 21.3 mm to (21.9, 31.9), turned to 270 degrees
- moved Y2 18.5 mm to (28.0, 34.0), turned to 180 degrees
- moved IC4 18.2 mm to (48.0, 25.3), turned to 90 degrees
- moved R1 17.7 mm to (38.5, 39.5)
- moved J1 15.4 mm to (64.1, 32.4), turned to 270 degrees
- moved R2 13.5 mm to (36.0, 39.5)
- moved R3 10.1 mm to (33.5, 39.5)
- moved IC2 7.10 mm to (24.0, 40.0), turned to 90 degrees
- moved IC1 4.01 mm to (48.0, 40.0)
- moved BAT1 1.41 mm to (10.0, 30.0)
Connections:
- new net N$6: IC5.24
- net A1: now also IC5.14; no longer IC4.14
- net A2: now also IC4.14; no longer IC5.14
- net B1: now also IC5.16; no longer IC4.16
- net B2: now also IC4.16; no longer IC5.16
- net C1: now also IC5.20; no longer IC4.20
- net C2: now also IC4.20; no longer IC5.20
- net D1: now also IC5.23; no longer IC4.23
- net D2: now also IC4.23; no longer IC5.23
- net DIG0: now also IC5.2; no longer IC4.2
- net DIG1: now also IC5.11; no longer IC4.11
- net DIG10: now also IC4.6; no longer IC5.6
- net DIG11: now also IC4.7; no longer IC5.7
- net DIG12: now also IC4.3; no longer IC5.3
- net DIG13: now also IC4.10; no longer IC5.10
- net DIG14: now also IC4.5; no longer IC5.5
- net DIG15: now also IC4.8; no longer IC5.8
- net DIG2: now also IC5.6; no longer IC4.6
- net DIG3: now also IC5.7; no longer IC4.7
- net DIG4: now also IC5.3; no longer IC4.3
- net DIG5: now also IC5.10; no longer IC4.10
- net DIG6: now also IC5.5; no longer IC4.5
- net DIG7: now also IC5.8; no longer IC4.8
- net DIG8: now also IC4.2; no longer IC5.2
- net DIG9: now also IC4.11; no longer IC5.11
- net DP1: now also IC5.22; no longer IC4.22
- net DP2: now also IC4.22; no longer IC5.22
- net E1: now also IC5.21; no longer IC4.21
- net E2: now also IC4.21; no longer IC5.21
- net F1: now also IC5.15; no longer IC4.15
- net F2: now also IC4.15; no longer IC5.15
- net G1: now also IC5.17; no longer IC4.17
- net G2: now also IC4.17; no longer IC5.17
- net MOSI/SDA: now also IC1.5
- net N$11: now also IC5.18; no longer IC4.18
- net N$12: now also IC4.18; no longer IC5.18
- net RST: now also IC1.1
- net SCK/SCL: now also IC1.7
