File: hardware/tick-mk-4.6.3.sch (EAGLE design)
At the start: 33 parts, among them IC1 ATMEGA328P, IC2 DS3231, IC3 L7805, Y1 16MHz

Commit message: think i'm done fiddling
Parts:
- JP1: value FTDI_CONNJST_PH_VERT_PTH -> FTDI_CONNJST_PH_VERT_PTH_LESSSILK; device A_butts:FTDI_CONNJST_PH_VERT_PTH -> A_butts:FTDI_CONNJST_PH_VERT_PTH_LESSSILK
- S1: value SPST-NO-TACT6MM-SMD -> SPST-NO-TACT6MM-PTH-SMALL-PADS; device A_butts:SPST-NO-TACT6MM-SMD -> A_butts:SPST-NO-TACT6MM-PTH-SMALL-PADS
Changed lines of the file:
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@@
 <part name="C5" library="A_butts" deviceset="CAPACITOR-POLARIZED" device="E2-5" value="10uF"/>
 <part name="SUPPLY1" library="A_butts" deviceset="VCC" device=""/>
-<part name="JP1" library="A_butts" deviceset="FTDI_CONN" device="JST_PH_VERT_PTH" value="FTDI_CONNJST_PH_VERT_PTH"/>
+<part name="JP1" library="A_butts" deviceset="FTDI_CONN" device="JST_PH_VERT_PTH_LESSSILK" value="FTDI_CONNJST_PH_VERT_PTH_LESSSILK"/>
 <part name="SUPPLY2" library="A_butts" deviceset="VCC" device=""/>
 <part name="GND3" library="A_butts" deviceset="GND" device=""/>
 <part name="C8" library="A_butts" deviceset="CAPACITOR-CERAMIC" device="025-024X044" value="0.1uF"/>
 <part name="IC2" library="A_butts" deviceset="DS3231" device=""/>
-<part name="S1" library="A_butts" deviceset="SPST-NO-TACT" device="6MM-SMD"/>
+<part name="S1" library="A_butts" deviceset="SPST-NO-TACT" device="6MM-PTH-SMALL-PADS" value="SPST-NO-TACT6MM-PTH-SMALL-PADS"/>
 <part name="GND6" library="A_butts" deviceset="GND" device=""/>
 </parts>
