File: hardware/tick-mk-4.6.4.sch (EAGLE design)
At the start: 33 parts, among them IC1 ATMEGA328P, IC2 DS3231, IC3 L7805, Y1 16MHz

Commit message: headers swapped, layout de-fucked a bit more
Parts:
- added C9: 0.1uF, A_butts:CAPACITOR-CERAMIC025-024X044
- JP1: value FTDI_CONNJST_PH_VERT_PTH_LESSSILK -> FTDI_CONNFLIPPER; device A_butts:FTDI_CONNJST_PH_VERT_PTH_LESSSILK -> A_butts:FTDI_CONNFLIPPER
- renumbered S1 to RESET
Connections:
- new net N$1: C9.2, IC1.AREF
- net GND: now also C9.1
Changed lines of the file:
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@@
 <part name="C5" library="A_butts" deviceset="CAPACITOR-POLARIZED" device="E2-5" value="10uF"/>
 <part name="SUPPLY1" library="A_butts" deviceset="VCC" device=""/>
-<part name="JP1" library="A_butts" deviceset="FTDI_CONN" device="JST_PH_VERT_PTH_LESSSILK" value="FTDI_CONNJST_PH_VERT_PTH_LESSSILK"/>
+<part name="JP1" library="A_butts" deviceset="FTDI_CONN" device="FLIPPER" value="FTDI_CONNFLIPPER"/>
 <part name="SUPPLY2" library="A_butts" deviceset="VCC" device=""/>
 <part name="GND3" library="A_butts" deviceset="GND" device=""/>
 <part name="C8" library="A_butts" deviceset="CAPACITOR-CERAMIC" device="025-024X044" value="0.1uF"/>
 <part name="IC2" library="A_butts" deviceset="DS3231" device=""/>
-<part name="S1" library="A_butts" deviceset="SPST-NO-TACT" device="6MM-PTH-SMALL-PADS" value="SPST-NO-TACT6MM-PTH-SMALL-PADS"/>
+<part name="RESET" library="A_butts" deviceset="SPST-NO-TACT" device="6MM-PTH-SMALL-PADS" value="SPST-NO-TACT6MM-PTH-SMALL-PADS"/>
 <part name="GND6" library="A_butts" deviceset="GND" device=""/>
+<part name="C9" library="A_butts" deviceset="CAPACITOR-CERAMIC" device="025-024X044" value="0.1uF"/>
+<part name="GND7" library="A_butts" deviceset="GND" device=""/>
 </parts>
 <sheets>
@@
 <instance part="C8" gate="G$1" x="203.2" y="139.7"/>
 <instance part="IC2" gate="G$1" x="124.46" y="121.92"/>
-<instance part="S1" gate="G$1" x="228.6" y="137.16"/>
+<instance part="RESET" gate="G$1" x="228.6" y="137.16"/>
 <instance part="GND6" gate="1" x="236.22" y="132.08"/>
+<instance part="C9" gate="G$1" x="2.54" y="132.08" rot="MR180"/>
+<instance part="GND7" gate="1" x="2.54" y="121.92"/>
 </instances>
 <busses>
@@
 </segment>
 <segment>
-<pinref part="S1" gate="G$1" pin="2"/>
+<pinref part="RESET" gate="G$1" pin="2"/>
 <wire x1="233.68" y1="137.16" x2="236.22" y2="137.16" width="0.1524" layer="91"/>
 <pinref part="GND6" gate="1" pin="GND"/>
 <wire x1="236.22" y1="137.16" x2="236.22" y2="134.62" width="0.1524" layer="91"/>
 </segment>
+<segment>
+<pinref part="C9" gate="G$1" pin="1"/>
+<pinref part="GND7" gate="1" pin="GND"/>
+<wire x1="2.54" y1="124.46" x2="2.54" y2="127" width="0.1524" layer="91"/>
+</segment>
 </net>
 <net name="RST" class="0">
@@
 <wire x1="220.98" y1="137.16" x2="223.52" y2="137.16" width="0.1524" layer="91"/>
 <label x="220.98" y="137.16" size="1.27" layer="95" rot="R180" xref="yes"/>
-<pinref part="S1" gate="G$1" pin="1"/>
+<pinref part="RESET" gate="G$1" pin="1"/>
 </segment>
 </net>
@@
 </segment>
 </net>
+<net name="N$1" class="0">
+<segment>
+<pinref part="IC1" gate="G$1" pin="AREF"/>
+<wire x1="35.56" y1="139.7" x2="2.54" y2="139.7" width="0.1524" layer="91"/>
+<wire x1="2.54" y1="139.7" x2="2.54" y2="137.16" width="0.1524" layer="91"/>
+<pinref part="C9" gate="G$1" pin="2"/>
+</segment>
+</net>
