File: hardware/tick-box-1591b-shield-mk-1.0.sch (EAGLE design)
At the start: 15 parts, among them IC1 DS3231, U1 ARDUINO_SHIELDINSIDER

Commit message: clocks are hard, some more stabs
Parts:
- U1: value ARDUINO_SHIELDINSIDER -> ARDUINO_SHIELDNOOUTLINE_NOHOLES; device A_butts:ARDUINO_SHIELDINSIDER -> A_butts:ARDUINO_SHIELDNOOUTLINE_NOHOLES
Changed lines of the file:
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@@
 <part name="H3" library="A_butts" deviceset="HOLE" device="#2" value="HOLE#2"/>
 <part name="H4" library="A_butts" deviceset="HOLE" device="#2" value="HOLE#2"/>
-<part name="U1" library="A_butts" deviceset="ARDUINO_SHIELD" device="INSIDER"/>
+<part name="U1" library="A_butts" deviceset="ARDUINO_SHIELD" device="NOOUTLINE_NOHOLES" value="ARDUINO_SHIELDNOOUTLINE_NOHOLES"/>
 <part name="GND1" library="A_butts" deviceset="GND" device=""/>
 </parts>
