File: hardware/tick-box-1591A-mk-2.0.brd (EAGLE design)
At the start: 78 x 42 mm, 26 parts, among them IC1 ATMEGA328P, IC2 DS3231, IC3 LM2931, Y1 16MHz

Commit message: alskdfjasdlfj
Parts:
- added C6: 0.1uF, A_butts:C025-024X044
- added D1: 1N4007, A_butts:DIODE-10.16MM
- C4: device A_butts:C025-024X044 -> A_butts:E2-4
- C5: value 10uF -> 47uF; device A_butts:C025-024X044 -> A_butts:E2-4
- IC3: device A_butts:SO08 -> A_butts:TO-92-AMMO
- moved RESET 23.1 mm to (75.5, 24.5), turned to 270 degrees
- moved C4 6.70 mm to (38.7, 2.30), flipped to the bottom, turned to 0 degrees
- moved IC3 5.92 mm to (44.7, 2.80), flipped to the bottom, turned to 180 degrees
- moved C5 5.20 mm to (51.2, 2.30), flipped to the bottom, turned to 180 degrees
- moved C3 5.15 mm to (51.5, 35.5), flipped to the top
- moved AVR_ISP 1.00 mm to (71.0, 34.0)
- moved C7 0.50 mm to (67.0, 21.9)
- moved C8 0.50 mm to (67.0, 26.9), turned to 270 degrees
- moved Y1 0.50 mm to (70.5, 24.5)
- turned R1 to 0 degrees
Connections:
- new net N$3: D1.A, F1.2, TVS1.P$2
- net GND: now also C3.2, C4.-, C5.-; no longer C4.2, C5.2, IC3.3, IC3.4, IC3.5, IC3.6, IC3.7
- net N$5: now also C4.+, D1.C, IC3.1; no longer C4.1, F1.2, IC3.8, TVS1.P$2
- net N$7: now also C6.2; no longer C3.2
- net RST: now also C6.1; no longer C3.1
- net VCC: now also C3.1, C5.+, IC3.3; no longer C5.1, IC3.1
Routing:
- net RST: track 0.00 -> 110.5 mm, vias 0 -> 1
- net VCC: track 55.8 -> 86.6 mm
- net SDA: track 0.00 -> 26.6 mm
- net VBAT: track 0.00 -> 24.0 mm, vias 0 -> 1
- net D9: track 69.0 -> 92.2 mm
- net SCL: track 0.00 -> 23.1 mm
- net D13/SCK: track 0.00 -> 19.9 mm
- net D10: track 42.1 -> 59.7 mm, vias 2 -> 3
- net D5: track 56.3 -> 71.4 mm, vias 2 -> 3
- net D11/MOSI: track 0.00 -> 13.5 mm
- net D12/MISO: track 0.00 -> 13.5 mm
- net D7: track 70.2 -> 82.3 mm, vias 2 -> 3
- net D8: track 60.7 -> 70.9 mm, vias 1 -> 2
- net N$5: track 19.0 -> 9.91 mm
- net D6: track 69.6 -> 78.0 mm, vias 3 -> 4
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