File: hardware/tick-box-1591A-mk-2.0.sch (EAGLE design)
At the start: 26 parts, among them IC1 ATMEGA328P, IC2 DS3231, IC3 LM2931, Y1 16MHz

Commit message: alskdfjasdlfj
Parts:
- added C6: 0.1uF, A_butts:CAPACITOR-CERAMIC025-024X044
- added D1: 1N4007, A_butts:DIODEPTH-10.68MM
- C4: device A_butts:CAPACITOR-CERAMIC025-024X044 -> A_butts:CAPACITOR-POLARIZEDE2-4
- C5: value 10uF -> 47uF; device A_butts:CAPACITOR-CERAMIC025-024X044 -> A_butts:CAPACITOR-POLARIZEDE2-4
- IC3: device A_butts:LM2931-FIXED -> A_butts:V_REG_78XXTO-92-INLINE
Connections:
- new net N$3: D1.A, F1.2, TVS1.2
- net GND: now also C3.2, C4.-, C5.-; no longer C4.2, C5.2
- net N$5: now also C4.+, D1.C; no longer C4.1, F1.2, TVS1.2
- net N$7: now also C6.2; no longer C3.2
- net RST: now also C6.1; no longer C3.1
- net VCC: now also C3.1, C5.+; no longer C5.1
Other:
- moved on the sheet: C3
