File: hardware/tick-box-1591A-mk-3.1.brd (EAGLE design)
At the start: 80 x 42 mm, 12 parts, among them IC2 DS3231, U1 ARDUINO_PRO_MINIMINE

Commit message: alskdfjasdlfj
Parts:
- removed DC_IN: M02PTH, A_butts:1X02
- added PWR1, PWR2: M02PTH-CENTERED, A_butts:1X02-CENTER
- C1: device A_butts:C0603 -> A_butts:C025-024X044
- U1: value ARDUINO_PRO_MINIMINE -> ARDUINO_PRO_MINI_TICK; device A_butts:ARDUINO_PRO_MINI_MINE -> A_butts:ARDUINO_PRO_MINI_TICK
- moved U1 25.2 mm to (14.8, 28.0)
- moved C1 15.4 mm to (76.4, 19.8), turned to 180 degrees
- moved RTC_BATT 4.50 mm to (59.5, 30.0)
- moved H1 4.00 mm to (7.00, 2.50)
- moved H2 4.00 mm to (7.00, 39.5)
- moved H3 4.00 mm to (73.0, 2.50)
- moved H4 4.00 mm to (73.0, 39.5)
- moved IC2 1.58 mm to (72.0, 27.0), turned to 0 degrees
- moved DISPLAY1 0.50 mm to (40.0, 28.0)
- moved DISPLAY2 0.50 mm to (60.0, 11.5)
- moved DISPLAY3 0.50 mm to (20.0, 11.5)
Connections:
- net A0: now also U1.A0; no longer U1.17
- net A1: now also U1.A1; no longer U1.18
- net A2: now also U1.A2; no longer U1.19
- net D10: now also U1.10; no longer U1.13
- net D2: now also DISPLAY1.P$14, DISPLAY2.5, DISPLAY3.14, U1.2; no longer DISPLAY1.P$10, DISPLAY2.15, DISPLAY3.13, U1.5
- net D3: now also U1.3; no longer U1.6
- net D4: now also DISPLAY1.P$10, DISPLAY2.15, DISPLAY3.13, U1.4; no longer DISPLAY1.P$14, DISPLAY2.5, DISPLAY3.14, U1.7
- net D5: now also U1.5; no longer U1.8
- net D6: now also U1.6; no longer U1.9
- net D7: now also U1.7; no longer U1.10
- net D8: now also U1.8; no longer U1.11
- net D9: now also U1.9; no longer U1.12
- net GND: now also PWR1.2, PWR2.2, U1.GND@1, U1.GND@2; no longer DC_IN.1, U1.23, U1.4, U1.BLK, U1.GND
- net RAW: now also PWR1.1, PWR2.1, U1.RAW; no longer DC_IN.2, U1.24
- net RST: now also U1.RST@1, U1.RST@2; no longer U1.22, U1.3, U1.GRN
- net VCC: no longer U1.21
Routing:
- net VCC: track 0.00 -> 88.4 mm, vias 0 -> 1
- net A2: track 0.00 -> 73.5 mm, vias 0 -> 1
- net SCL: track 0.00 -> 64.6 mm
- net RAW: track 0.00 -> 64.1 mm
- net SDA: track 0.00 -> 60.0 mm
- net A1: track 0.00 -> 59.7 mm, vias 0 -> 1
- net D10: track 0.00 -> 48.4 mm
- net A0: track 0.00 -> 31.6 mm, vias 0 -> 1
- net VBAT: track 0.00 -> 8.94 mm, vias 0 -> 1
Other:
- board text added: "+"
- board text added: "-"
