File: hardware/tick-box-1591A-mk-3.1.sch (EAGLE design)
At the start: 12 parts, among them IC2 DS3231, U1 ARDUINO_PRO_MINIMINE

Commit message: alskdfjasdlfj
Parts:
- removed DC_IN: M02PTH, A_butts:M02PTH
- added PWR1, PWR2: M02PTH-CENTERED, A_butts:M02PTH-CENTERED
- C1: device A_butts:CAPACITOR-CERAMICC0603 -> A_butts:CAPACITOR-CERAMIC025-024X044
- U1: value ARDUINO_PRO_MINIMINE -> ARDUINO_PRO_MINI_TICK; device A_butts:ARDUINO_PRO_MINIMINE -> A_butts:ARDUINO_PRO_MINI_TICK
Connections:
- net D2: now also DISPLAY1.DIG1, DISPLAY2.E, DISPLAY3.A; no longer DISPLAY1.DIG3, DISPLAY2.G, DISPLAY3.C
- net D4: now also DISPLAY1.DIG3, DISPLAY2.G, DISPLAY3.C; no longer DISPLAY1.DIG1, DISPLAY2.E, DISPLAY3.A
- net GND: now also PWR1.2, PWR2.2; no longer DC_IN.1
- net RAW: now also PWR1.1, PWR2.1; no longer DC_IN.2
