File: hardware/tick-box-1591A-mk-2.1.brd (EAGLE design)
At the start: 80 x 42 mm, 13 parts, among them IC2 DS3231, U1 ARDUINO_PRO_MINI_TICK

Commit message: more attempts at a hammond 1591A sized clock
Parts:
- removed PWR1, PWR2: M02PTH-CENTERED, A_butts:1X02-CENTER
- removed U1: ARDUINO_PRO_MINI_TICK, A_butts:ARDUINO_PRO_MINI_TICK
- added AVR_ISP: AVR_SPI_PRG_6PTH, A_butts:2X3
- added C2, C3, C6: 0.1uF, A_butts:C025-024X044
- added C4: 10uF, A_butts:E2-4
- added C5: 47uF, A_butts:E2-4
- added C7, C8: 22pF, A_butts:C025-024X044
- added D1: 1N4007, A_butts:DIODE-10.16MM
- added DC_IN: M02PTH, A_butts:1X02
- added F1: 250mA, A_butts:PTC-PTH-5.08MM
- added IC1: ATMEGA328P, A_butts:DIL28-3
- added IC3: LM2931, A_butts:TO-92-AMMO
- added JP1: FTDI_CONNFLIPPER, A_butts:FTDI_CONN_FLIP
- added R1: 10k, A_butts:RESISTOR-AXIAL-PTH-6.35MM
- added RESET: SPST-NO-TACT3MM-PTH-SMALL-PADS, A_butts:DTS-3-SMALL-PADS
- added TVS1: SA5.0CA, A_butts:DO-41-TVS-BI-10.16MM
- added Y1: 16MHz, A_butts:HC49U-V
- RTC_BATT: value CR2032 -> CR1225; device A_butts:BATTCON_20MM_MINE -> A_butts:BATTCON_12MM_PTH_TOPLOAD
- moved IC2 58.0 mm to (14.0, 25.0), flipped to the top, turned to 270 degrees
- moved RTC_BATT 53.5 mm to (6.00, 28.0), flipped to the bottom
- moved C1 32.4 mm to (44.1, 20.4)
- moved H4 6.50 mm to (66.5, 39.5)
- moved H2 4.50 mm to (11.5, 39.5)
- moved H3 2.00 mm to (71.0, 2.50)
- moved DISPLAY1 1.00 mm to (39.0, 28.0)
- moved DISPLAY2 1.00 mm to (59.0, 11.5)
- moved DISPLAY3 1.00 mm to (19.0, 11.5)
Connections:
- removed net RAW: PWR1.1, PWR2.1, U1.RAW
- new net D11/MOSI: AVR_ISP.4, IC1.17
- new net D12/MISO: AVR_ISP.1, IC1.18
- new net D13/SCK: AVR_ISP.3, IC1.19
- new net N$1: C7.1, IC1.10, Y1.1
- new net N$2: C8.1, IC1.9, Y1.2
- new net N$3: D1.A, F1.P$2, TVS1.P$2
- new net N$4: DC_IN.2, F1.P$1
- new net N$5: C4.+, D1.C, IC3.1
- new net N$7: C6.2, JP1.DTR
- new net RX: IC1.2, JP1.RXI
- new net TX: IC1.3, JP1.TXO
- net A0: now also IC1.23; no longer U1.A0
- net A1: now also IC1.24; no longer U1.A1
- net A2: now also IC1.25; no longer U1.A2
- net D10: now also IC1.16; no longer U1.10
- net D2: now also DISPLAY1.P$10, DISPLAY2.15, DISPLAY3.13, IC1.4; no longer DISPLAY1.P$14, DISPLAY2.5, DISPLAY3.14, U1.2
- net D3: now also IC1.5; no longer U1.3
- net D4: now also DISPLAY1.P$14, DISPLAY2.5, DISPLAY3.14, IC1.6; no longer DISPLAY1.P$10, DISPLAY2.15, DISPLAY3.13, U1.4
- net D5: now also IC1.11; no longer U1.5
- net D6: now also IC1.12; no longer U1.6
- net D7: now also IC1.13; no longer U1.7
- net D8: now also IC1.14; no longer U1.8
- net D9: now also IC1.15; no longer U1.9
- net GND: now also AVR_ISP.6, C2.2, C3.2, C4.-, C5.-, C7.2, C8.2, DC_IN.1, IC1.22, IC1.8, IC3.2, JP1.CTS, JP1.GND, RESET.2, RTC_BATT.-, TVS1.P$1; no longer PWR1.2, PWR2.2, RTC_BATT.BOTTOM, U1.GND@1, U1.GND@2
- net RST: now also AVR_ISP.5, C6.1, IC1.1, R1.P$2, RESET.1; no longer U1.RST@1, U1.RST@2
- net SCL: now also IC1.28; no longer U1.A5
- net SDA: now also IC1.27; no longer U1.A4
- net VBAT: now also RTC_BATT.+; no longer RTC_BATT.TOP@2
- net VCC: now also AVR_ISP.2, C2.1, C3.1, C5.+, IC1.20, IC1.7, IC3.3, JP1.VCC, R1.P$1; no longer U1.VCC
Routing:
- net A1: track 111.2 -> 0.00 mm, vias 2 -> 0
- net A2: track 109.5 -> 0.00 mm, vias 3 -> 0
- net A0: track 99.4 -> 0.00 mm, vias 2 -> 0
- net RST: track 90.2 -> 0.00 mm, vias 1 -> 0
- net VCC: track 88.0 -> 0.00 mm, vias 1 -> 0
- net D10: track 86.5 -> 0.00 mm, vias 1 -> 0
- net D9: track 83.6 -> 0.00 mm, vias 4 -> 0
- net D5: track 79.9 -> 0.00 mm, vias 2 -> 0
- net D7: track 76.1 -> 0.00 mm, vias 4 -> 0
- net D6: track 75.3 -> 0.00 mm, vias 3 -> 0
- net D8: track 72.0 -> 0.00 mm, vias 4 -> 0
- net D2: track 68.6 -> 0.00 mm, vias 3 -> 0
- net D4: track 65.5 -> 0.00 mm, vias 3 -> 0
- net SCL: track 64.6 -> 0.00 mm
- net RAW: track 64.1 -> 0.00 mm
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- removed copper zone on layer 16, net GND
Other:
- board size 80 x 42 mm -> 78 x 42 mm
- board text removed: "+"
- board text removed: "-"
