File: hardware/tick-box-1591A-mk-2.2.sch (EAGLE design)
At the start: 26 parts, among them IC1 ATMEGA328P, IC2 DS3231, IC3 LM2931, Y1 16MHz

Commit message: layout done
Parts:
- removed PWR1: DCBARRELSMT, A_butts:DCBARRELSMT
- added PWR: M02PTH-CENTERED, A_butts:M02PTH-CENTERED
- added Y2: 32.768kHz, A_butts:CRYSTALTC26H
- C3: value 0.1uF -> 1uF
- C4: device A_butts:CAPACITOR-POLARIZEDE2-4 -> A_butts:CAPACITOR-POLARIZEDE2-5
- C5: device A_butts:CAPACITOR-POLARIZEDE2-4 -> A_butts:CAPACITOR-POLARIZEDE2.5-6
- IC2: value DS3231 -> DS1307; device A_butts:DS3231 -> A_butts:DS1307
- RTC_BATT: value CR2032 -> CR1225
Connections:
- new net N$6: IC2.X2, Y2.1
- new net N$8: IC2.X1, Y2.2
- net GND: now also PWR.1; no longer PWR1.GND
- net N$4: now also PWR.2; no longer PWR1.PWR
- net RST: no longer IC2.!RST
Changed lines of the file:
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@@
 <setting verticaltext="up"/>
 </settings>
-<grid distance="100" unitdist="mil" unit="mil" style="lines" multiple="1" display="yes" altdistance="1" altunitdist="mil" altunit="mil"/>
+<grid distance="100" unitdist="mil" unit="mil" style="lines" multiple="1" display="yes" altdistance="2" altunitdist="mil" altunit="mil"/>
 <layers>
 <layer number="1" name="Top" color="4" fill="1" visible="yes" active="no"/>
@@
 <part name="C2" library="A_butts" deviceset="CAPACITOR-CERAMIC" device="025-024X044" value="0.1uF"/>
 <part name="SUPPLY7" library="A_butts" deviceset="VCC" device=""/>
-<part name="IC2" library="A_butts" deviceset="DS3231" device=""/>
 <part name="DISPLAY1" library="A_butts" deviceset="7SEG_4DIGIT_COLON" device="14.2MM-CC-NS" value="7SEG_4DIGIT_COLON14.2MM-CC-NS"/>
 <part name="GND2" library="A_butts" deviceset="GND" device=""/>
@@
 <part name="TVS1" library="A_butts" deviceset="TVS" device="DO-41-10.16MM" value="SA5.0CA"/>
 <part name="GND6" library="A_butts" deviceset="GND" device=""/>
-<part name="C4" library="A_butts" deviceset="CAPACITOR-POLARIZED" device="E2-4" value="10uF"/>
-<part name="C5" library="A_butts" deviceset="CAPACITOR-POLARIZED" device="E2-4" value="47uF"/>
+<part name="C4" library="A_butts" deviceset="CAPACITOR-POLARIZED" device="E2-5" value="10uF"/>
+<part name="C5" library="A_butts" deviceset="CAPACITOR-POLARIZED" device="E2.5-6" value="47uF"/>
 <part name="IC3" library="A_butts" deviceset="V_REG_78XX" device="TO-92-INLINE" value="LM2931"/>
 <part name="D1" library="A_butts" deviceset="DIODE" device="PTH-10.68MM" value="1N4007"/>
 <part name="GND12" library="A_butts" deviceset="GND" device=""/>
-<part name="C3" library="A_butts" deviceset="CAPACITOR-CERAMIC" device="025-024X044" value="0.1uF"/>
+<part name="C3" library="A_butts" deviceset="CAPACITOR-CERAMIC" device="025-024X044" value="1uF"/>
 <part name="SUPPLY9" library="A_butts" deviceset="VCC" device=""/>
 <part name="C6" library="A_butts" deviceset="CAPACITOR-CERAMIC" device="025-024X044" value="0.1uF"/>
 <part name="Y1" library="A_butts" deviceset="RESONATOR" device="PTH" value="16MHz"/>
-<part name="PWR1" library="A_butts" deviceset="DCBARREL" device="SMT" value="DCBARRELSMT"/>
-<part name="RTC_BATT" library="A_butts" deviceset="BATTERY" device="12PTH_TOPLOAD" value="CR2032"/>
+<part name="RTC_BATT" library="A_butts" deviceset="BATTERY" device="12PTH_TOPLOAD" value="CR1225"/>
+<part name="IC2" library="A_butts" deviceset="DS1307" device=""/>
+<part name="Y2" library="A_butts" deviceset="CRYSTAL" device="TC26H" value="32.768kHz"/>
+<part name="PWR" library="A_butts" deviceset="M02" device="PTH-CENTERED" value="M02PTH-CENTERED"/>
 </parts>
 <sheets>
@@
 <instance part="C1" gate="G$1" x="132.08" y="48.26"/>
 <instance part="SUPPLY3" gate="G$1" x="132.08" y="55.88"/>
-<instance part="SUPPLY6" gate="G$1" x="109.22" y="129.54"/>
-<instance part="GND9" gate="1" x="109.22" y="111.76"/>
+<instance part="SUPPLY6" gate="G$1" x="129.54" y="142.24"/>
+<instance part="GND9" gate="1" x="121.92" y="99.06"/>
 <instance part="GND10" gate="1" x="142.24" y="38.1"/>
 <instance part="C2" gate="G$1" x="142.24" y="48.26"/>
 <instance part="SUPPLY7" gate="G$1" x="142.24" y="55.88"/>
-<instance part="IC2" gate="G$1" x="124.46" y="121.92"/>
 <instance part="DISPLAY1" gate="G$1" x="88.9" y="71.12"/>
 <instance part="GND2" gate="1" x="139.7" y="99.06"/>
@@
 <instance part="C6" gate="G$1" x="190.5" y="157.48" rot="R90"/>
 <instance part="Y1" gate="G$1" x="12.7" y="121.92"/>
-<instance part="PWR1" gate="G$1" x="165.1" y="93.98"/>
 <instance part="RTC_BATT" gate="G$1" x="139.7" y="109.22" rot="MR270"/>
+<instance part="IC2" gate="G$1" x="121.92" y="119.38"/>
+<instance part="Y2" gate="G$1" x="119.38" y="142.24" rot="MR0"/>
+<instance part="PWR" gate="G$1" x="157.48" y="91.44"/>
 </instances>
 <busses>
@@
 <pinref part="SUPPLY3" gate="G$1" pin="VCC"/>
 <wire x1="132.08" y1="55.88" x2="132.08" y2="53.34" width="0.1524" layer="91"/>
-</segment>
-<segment>
-<pinref part="SUPPLY6" gate="G$1" pin="VCC"/>
-<wire x1="109.22" y1="129.54" x2="109.22" y2="127" width="0.1524" layer="91"/>
-<wire x1="109.22" y1="127" x2="111.76" y2="127" width="0.1524" layer="91"/>
-<pinref part="IC2" gate="G$1" pin="VCC"/>
 </segment>
 <segment>
@@
 <wire x1="152.4" y1="55.88" x2="152.4" y2="53.34" width="0.1524" layer="91"/>
 </segment>
+<segment>
+<pinref part="IC2" gate="G$1" pin="VCC"/>
+<pinref part="SUPPLY6" gate="G$1" pin="VCC"/>
+<wire x1="129.54" y1="137.16" x2="129.54" y2="142.24" width="0.1524" layer="91"/>
+</segment>
 </net>
 <net name="GND" class="0">
@@
 </segment>
 <segment>
-<pinref part="GND9" gate="1" pin="GND"/>
-<wire x1="109.22" y1="116.84" x2="109.22" y2="114.3" width="0.1524" layer="91"/>
-<wire x1="109.22" y1="116.84" x2="111.76" y2="116.84" width="0.1524" layer="91"/>
-<pinref part="IC2" gate="G$1" pin="GND"/>
-</segment>
-<segment>
 <pinref part="C2" gate="G$1" pin="2"/>
 <pinref part="GND10" gate="1" pin="GND"/>
@@
 </segment>
 <segment>
-<wire x1="170.18" y1="91.44" x2="170.18" y2="78.74" width="0.1524" layer="91"/>
+<wire x1="170.18" y1="93.98" x2="170.18" y2="78.74" width="0.1524" layer="91"/>
 <wire x1="170.18" y1="78.74" x2="185.42" y2="78.74" width="0.1524" layer="91"/>
 <wire x1="185.42" y1="78.74" x2="205.74" y2="78.74" width="0.1524" layer="91"/>
@@
 <wire x1="231.14" y1="78.74" x2="231.14" y2="83.82" width="0.1524" layer="91"/>
 <wire x1="218.44" y1="78.74" x2="218.44" y2="88.9" width="0.1524" layer="91"/>
-<wire x1="167.64" y1="91.44" x2="170.18" y2="91.44" width="0.1524" layer="91"/>
+<wire x1="167.64" y1="93.98" x2="170.18" y2="93.98" width="0.1524" layer="91"/>
 <pinref part="TVS1" gate="G$1" pin="1"/>
 <wire x1="185.42" y1="81.28" x2="185.42" y2="78.74" width="0.1524" layer="91"/>
@@
 <pinref part="C5" gate="G$1" pin="-"/>
 <pinref part="IC3" gate="G$1" pin="GND"/>
-<pinref part="PWR1" gate="G$1" pin="GND"/>
+<pinref part="PWR" gate="G$1" pin="1"/>
 </segment>
 <segment>
@@
 <wire x1="12.7" y1="111.76" x2="12.7" y2="114.3" width="0.1524" layer="91"/>
 </segment>
+<segment>
+<pinref part="IC2" gate="G$1" pin="GND"/>
+<pinref part="GND9" gate="1" pin="GND"/>
+<wire x1="121.92" y1="101.6" x2="121.92" y2="104.14" width="0.1524" layer="91"/>
+</segment>
 </net>
 <net name="RST" class="0">
@@
 </segment>
 <segment>
-<wire x1="106.68" y1="124.46" x2="111.76" y2="124.46" width="0.1524" layer="91"/>
-<label x="106.68" y="124.46" size="1.27" layer="95" rot="R180" xref="yes"/>
-<pinref part="IC2" gate="G$1" pin="!RST"/>
-</segment>
-<segment>
 <wire x1="162.56" y1="40.64" x2="162.56" y2="43.18" width="0.1524" layer="91"/>
 <label x="162.56" y="40.64" size="1.27" layer="95" rot="R270" xref="yes"/>
@@
 <label x="147.32" y="116.84" size="1.27" layer="95" xref="yes"/>
 <wire x1="139.7" y1="116.84" x2="137.16" y2="116.84" width="0.1524" layer="91"/>
-<pinref part="IC2" gate="G$1" pin="VBAT"/>
 <wire x1="139.7" y1="114.3" x2="139.7" y2="116.84" width="0.1524" layer="91"/>
 <junction x="139.7" y="116.84"/>
 <pinref part="RTC_BATT" gate="G$1" pin="+"/>
+<pinref part="IC2" gate="G$1" pin="VBAT"/>
 </segment>
 </net>
@@
 <pinref part="F1" gate="G$1" pin="1"/>
 <wire x1="167.64" y1="96.52" x2="172.72" y2="96.52" width="0.1524" layer="91"/>
-<pinref part="PWR1" gate="G$1" pin="PWR"/>
+<pinref part="PWR" gate="G$1" pin="2"/>
 </segment>
 </net>
 <net name="SDA" class="0">
 <segment>
-<label x="106.68" y="121.92" size="1.27" layer="95" rot="R180" xref="yes"/>
-<wire x1="106.68" y1="121.92" x2="111.76" y2="121.92" width="0.1524" layer="91"/>
+<label x="104.14" y="116.84" size="1.27" layer="95" rot="R180" xref="yes"/>
+<wire x1="104.14" y1="116.84" x2="106.68" y2="116.84" width="0.1524" layer="91"/>
 <pinref part="IC2" gate="G$1" pin="SDA"/>
 </segment>
@@
 <net name="SCL" class="0">
 <segment>
-<label x="106.68" y="119.38" size="1.27" layer="95" rot="R180" xref="yes"/>
-<wire x1="106.68" y1="119.38" x2="111.76" y2="119.38" width="0.1524" layer="91"/>
+<label x="104.14" y="121.92" size="1.27" layer="95" rot="R180" xref="yes"/>
+<wire x1="104.14" y1="121.92" x2="106.68" y2="121.92" width="0.1524" layer="91"/>
 <pinref part="IC2" gate="G$1" pin="SCL"/>
 </segment>
@@
 </segment>
 </net>
+<net name="N$6" class="0">
+<segment>
+<pinref part="IC2" gate="G$1" pin="X2"/>
+<pinref part="Y2" gate="G$1" pin="1"/>
+<wire x1="121.92" y1="142.24" x2="121.92" y2="137.16" width="0.1524" layer="91"/>
+</segment>
+</net>
+<net name="N$8" class="0">
+<segment>
+<pinref part="IC2" gate="G$1" pin="X1"/>
+<pinref part="Y2" gate="G$1" pin="2"/>
+<wire x1="116.84" y1="142.24" x2="116.84" y2="137.16" width="0.1524" layer="91"/>
+</segment>
+</net>
