File: hardware/tick-box-1591A-mk-2.2.brd (EAGLE design)
At the start: 92 x 42 mm, 26 parts, among them IC1 ATMEGA328P, IC2 DS3231, IC3 LM2931, Y1 16MHz

Commit message: layout done
Parts:
- removed PWR1: DCBARRELSMT, A_butts:DCJACK_2MM_SMT
- added PWR: M02PTH-CENTERED, A_butts:1X02-CENTER
- added Y2: 32.768kHz, A_butts:TC26H
- C3: value 0.1uF -> 1uF
- C4: device A_butts:E2-4 -> A_butts:E2-5
- C5: device A_butts:E2-4 -> A_butts:E2,5-6
- IC2: value DS3231 -> DS1307; device A_butts:SO16W -> A_butts:DIL08
- RTC_BATT: value CR2032 -> CR1225
- moved F1 65.9 mm to (89.0, 20.5), flipped to the bottom, turned to 90 degrees
- moved TVS1 53.9 mm to (79.0, 36.0), flipped to the bottom, turned to 180 degrees
- moved C3 48.9 mm to (78.8, 27.0), flipped to the bottom, turned to 270 degrees
- moved JP1 47.5 mm to (2.50, 21.0), flipped to the bottom, turned to 270 degrees
- moved RESET 44.5 mm to (75.0, 21.0), flipped to the bottom
- moved D1 43.5 mm to (79.0, 32.0), flipped to the bottom, turned to 180 degrees
- moved C4 42.8 mm to (89.0, 27.0), flipped to the bottom, turned to 180 degrees
- moved R1 36.7 mm to (34.0, 28.0), turned to 270 degrees
- moved C5 34.9 mm to (75.0, 27.0), flipped to the bottom
- moved C6 33.0 mm to (34.0, 22.0), turned to 180 degrees
- moved IC3 32.4 mm to (83.0, 27.0), flipped to the bottom
- moved C2 29.8 mm to (28.0, 30.5), turned to 270 degrees
- moved C1 22.3 mm to (59.0, 34.0)
- moved H1 10.5 mm to (3.00, 9.00)
- moved H2 10.5 mm to (89.0, 9.00)
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Connections:
- new net N$6: IC2.2, Y2.1
- new net N$8: IC2.1, Y2.2
- net GND: now also IC2.4, PWR.1; no longer IC2.10, IC2.11, IC2.12, IC2.13, IC2.5, IC2.6, IC2.7, IC2.8, IC2.9, PWR1.GND
- net N$4: now also PWR.2; no longer PWR1.PWR@1, PWR1.PWR@2
- net RST: no longer IC2.4
- net SCL: now also IC2.6; no longer IC2.16
- net SDA: now also IC2.5; no longer IC2.15
- net VBAT: now also IC2.3; no longer IC2.14
- net VCC: now also IC2.8; no longer IC2.2
Other:
- board size 92 x 42 mm -> 92 x 34 mm

Commit message: more layout tweaks for smt design
Parts:
- moved TVS1 10.0 mm to (79.0, 26.0)
- moved C3 8.02 mm to (78.2, 35.0), turned to 90 degrees
- moved C5 7.57 mm to (74.0, 34.5)
- moved IC3 7.50 mm to (83.0, 34.5)
- moved D1 2.00 mm to (79.0, 30.0)
- moved C4 1.41 mm to (88.0, 28.0), turned to 270 degrees
- turned C1 to 180 degrees
Routing:
- net VCC: track 0.00 -> 120.8 mm
- net RST: track 0.00 -> 54.3 mm
- net TX: track 0.00 -> 43.4 mm, vias 0 -> 1
- net RX: track 0.00 -> 40.3 mm
- net N$7: track 0.00 -> 32.4 mm
- net D12/MISO: track 0.00 -> 30.2 mm
- net D13/SCK: track 0.00 -> 29.8 mm, vias 0 -> 1
- net D9: track 0.00 -> 22.2 mm
- net D11/MOSI: track 0.00 -> 21.8 mm
- net N$3: track 0.00 -> 18.0 mm
- net VBAT: track 0.00 -> 17.7 mm
- net SDA: track 0.00 -> 17.4 mm
- net D10: track 0.00 -> 15.9 mm
- net SCL: track 0.00 -> 13.8 mm
- net N$5: track 0.00 -> 11.6 mm
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