File: hardware/tick-wifi-mk-1.0.brd (EAGLE design)
At the start: 100 x 64 mm, 39 parts, among them IC1 MAX7219, IC2 MAX7219, IC3 74HC125, IC4 LD1117 5V, IC5 LD1117 3V, Q1 MMBT2222, Q2 MMBT2222

Commit message: wip
Routing:
- net 5V: track 179.7 -> 0.00 mm, vias 6 -> 0
- net SEG_1C: track 111.1 -> 0.00 mm, vias 3 -> 0
- net SEG_1E: track 108.1 -> 0.00 mm, vias 4 -> 0
- net SEG_1G: track 107.3 -> 0.00 mm, vias 4 -> 0
- net SEG_1F: track 107.0 -> 0.00 mm, vias 4 -> 0
- net SEG_1A: track 92.7 -> 0.00 mm, vias 3 -> 0
- net SEG_1P: track 92.4 -> 0.00 mm
- net SEG_1B: track 87.9 -> 0.00 mm, vias 1 -> 0
- net SEG_1D: track 82.6 -> 0.00 mm, vias 3 -> 0
- net VIN: track 48.5 -> 0.00 mm
- net DIG_4: track 30.5 -> 0.00 mm
- net DIG_1: track 30.5 -> 0.00 mm
- net CTRL_LOAD: track 29.6 -> 0.00 mm, vias 2 -> 0
- net DISP_LOAD: track 28.3 -> 0.00 mm, vias 1 -> 0
- net CTRL_CLCK: track 27.6 -> 0.00 mm
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
Commit message: more wip
Parts:
- DIGIT1, DIGIT2, DIGIT3, DIGIT4: device A_butts:7SEG_1DIG_25.4MM_NOSILK -> a_parts:7SEG_1DIG_25.4MM_NOSILK
- DISPLAY1, DISPLAY2: value 7SEG_4DIGIT_COLON14.2MM-CC -> 7SEG_4DIGIT_COLON_APOS; device a_parts:7SEG_4DIG_0.56IN_14MM_ADAFRUIT -> a_parts:7SEG_4DIG_10MM
- F1: device A_butts:PTC-1210 -> a_parts:PTC-1210
- FRAME1: device A_butts:DUMMY -> a_parts:DUMMY
- PWR_IN: device A_butts:1X02-CENTER-R+ -> a_parts:1X02-CENTER-R+
- TVS1: device A_butts:SMA-DIODE-TVS-BIDIR -> a_parts:SMA-DIODE-TVS-BIDIR
- U$1: device A_butts:TICK_SYMBOL -> a_parts:TICK_SYMBOL
- U$2: device A_butts:COW_SMALL -> a_parts:COW_SMALL
- U$4: device A_butts:CC-BY-SA-4.0-NO-URL -> a_parts:CC-BY-SA-4.0-NO-URL
- moved U$4 87.6 mm to (76.1, 66.8)
- moved U$3 60.3 mm to (6.20, 63.3)
- moved U$2 35.3 mm to (57.7, 65.5)
- moved PWR_IN 22.3 mm to (92.6, 15.7)
- moved DIGIT1 8.00 mm to (86.0, 34.0)
- moved DIGIT2 8.00 mm to (62.0, 34.0)
- moved DIGIT3 8.00 mm to (38.0, 34.0)
- moved DIGIT4 8.00 mm to (14.0, 34.0)
- moved IC1 8.00 mm to (50.0, 34.0)
- moved R10 8.00 mm to (8.50, 45.5)
- moved R5 8.00 mm to (10.5, 45.5)
- moved U$1 8.00 mm to (50.0, 34.0)
- moved U1 8.00 mm to (13.0, 34.0)
- moved DISPLAY1 7.43 mm to (30.0, 9.00)
- moved DISPLAY2 7.43 mm to (70.0, 9.00)
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Connections:
- net DIG_10: now also DISPLAY2.2; no longer DISPLAY2.P$11
- net DIG_11: now also DISPLAY2.6; no longer DISPLAY2.P$10
- net DIG_12: now also DISPLAY2.8; no longer DISPLAY2.P$6
- net DIG_5: now also DISPLAY1.1; no longer DISPLAY1.P$14
- net DIG_6: now also DISPLAY1.2; no longer DISPLAY1.P$11
- net DIG_7: now also DISPLAY1.6; no longer DISPLAY1.P$10
- net DIG_8: now also DISPLAY1.8; no longer DISPLAY1.P$6
- net DIG_9: now also DISPLAY2.1; no longer DISPLAY2.P$14
- net GND: now also DISPLAY1.12, DISPLAY2.12; no longer DISPLAY1.P$7, DISPLAY2.P$7
- net N$3: now also DISPLAY1.4; no longer DISPLAY1.P$8
- net N$5: now also DISPLAY2.4; no longer DISPLAY2.P$8
- net SEG_2A: now also DISPLAY1.14, DISPLAY2.14; no longer DISPLAY1.P$13, DISPLAY2.P$13
- net SEG_2B: now also DISPLAY1.16, DISPLAY2.16; no longer DISPLAY1.P$9, DISPLAY2.P$9
- net SEG_2C: now also DISPLAY1.13, DISPLAY2.13; no longer DISPLAY1.P$4, DISPLAY2.P$4
- net SEG_2D: now also DISPLAY1.3, DISPLAY2.3; no longer DISPLAY1.P$2, DISPLAY2.P$2
- net SEG_2E: now also DISPLAY1.5, DISPLAY2.5; no longer DISPLAY1.P$1, DISPLAY2.P$1
- net SEG_2F: now also DISPLAY1.11, DISPLAY2.11; no longer DISPLAY1.P$12, DISPLAY2.P$12
- net SEG_2G: now also DISPLAY1.15, DISPLAY2.15; no longer DISPLAY1.P$5, DISPLAY2.P$5
- net SEG_2P: now also DISPLAY1.7, DISPLAY2.7; no longer DISPLAY1.P$3, DISPLAY2.P$3
Other:
- board size 100 x 64 mm -> 100 x 54 mm
