File: hardware/tick-wifi-mini-mk-1.3.brd (EAGLE design)
At the start: 50.8 x 22.9 mm, 15 parts, among them IC1 HT16K33, U1 Adafruit Feather HUZZAH ESP82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

Commit message: yet another attempt at a ht16k33 driver
Parts:
- removed U$1: (no value), a_parts:OSHWLOGO_TINY
- added A0, A1, A2: JUMPER-PAD-2-NOYES_SILK, a_parts:PAD-JUMPER-2-NO_YES_SILK
- added C2: 10uF, a_parts:C0805-TIGHTER
- added D2: PMEG2005CT, a_parts:SOT23
- added Q1, Q2: IRLML2502, a_parts:SOT23
- added R6, R7: 10K, a_parts:R0603-TIGHTER
- added U$3: (no value), a_parts:OSHWLOGO_TINY_SILKONLY
- C1: device a_parts:C0805 -> a_parts:C0603-TIGHTER
- D1: device a_parts:SOD123 -> a_parts:SOD323
- I2C: value M04-I2CJST-4-PH-VERT-CENTERED-I2C -> M04-I2CPTH-2MM-CENTERED; device a_parts:JST-4-PH-VERT-PTH-CENTERED-I2C -> a_parts:1X04-2MM-CENTERED-I2C
- R1, R2, R3: value 39K -> 47K; device a_parts:R0805 -> a_parts:R0603-TIGHTER
- R4, R5: value 4K7 -> 10K; device a_parts:R0805 -> a_parts:R0603-TIGHTER
- moved R1 35.3 mm to (7.62, 5.08)
- moved R2 34.1 mm to (7.62, 7.62)
- moved R3 33.7 mm to (7.62, 10.2)
- moved D1 30.2 mm to (11.4, 7.62), turned to 270 degrees
- moved C1 21.9 mm to (14.6, 11.4), turned to 270 degrees
- moved U$2 14.9 mm to (41.9, 11.4), turned to 90 degrees
- moved R5 12.2 mm to (4.45, 19.1), turned to 180 degrees
- moved U$4 11.1 mm to (43.8, 5.71), turned to 90 degrees
- moved I2C 9.23 mm to (42.4, 19.1), turned to 0 degrees
- moved R4 7.73 mm to (8.89, 19.1), turned to 180 degrees
- turned IC1 to 0 degrees
Connections:
- removed net SCL: I2C.4, IC1.26, R5.2, U1.SCL
- removed net SDA: I2C.3, IC1.27, R4.2, U1.SDA
- new net N$2: A0.1, R1.2
- new net N$3: A1.1, R2.2
- new net N$4: A2.1, R3.2
- new net SCL-3V3: Q1.2, R4.2, U1.SCL
- new net SCL-VCC: I2C.4, IC1.26, Q1.3, R6.2
- new net SDA-3V3: Q2.2, R5.2, U1.SDA
- new net SDA-VCC: I2C.3, IC1.27, Q2.3, R7.2
- new net VBAT: D2.1, U1.BAT
- new net VCC: C1.1, C2.1, D2.3, I2C.2, IC1.28, R6.1, R7.1
- new net VUSB: D2.2, U1.USB
- net 3.3V: now also Q1.1, Q2.1; no longer C1.1, I2C.2, IC1.28
- net GND: now also C2.2
- net SEG_A/A2: now also A2.2; no longer R3.2
- net SEG_B/A1/COL_A: now also A1.2; no longer R2.2
- net SEG_C/A0: now also A0.2; no longer R1.2
Routing:
- net SDA-VCC: track 0.00 -> 55.3 mm, vias 0 -> 4
- net VCC: track 0.00 -> 48.0 mm, vias 0 -> 2
- net SCL-VCC: track 0.00 -> 47.1 mm, vias 0 -> 3
- net DIG_1/ADDR_SEL: track 7.25 -> 31.9 mm, vias 0 -> 3
- net SDA: track 24.1 -> 0.00 mm, vias 1 -> 0
- net SEG_C/A0: track 19.7 -> 38.3 mm, vias 0 -> 1
- net SCL: track 17.1 -> 0.00 mm, vias 1 -> 0
- net SEG_E: track 0.00 -> 16.7 mm, vias 0 -> 1
- net SEG_D: track 0.00 -> 16.0 mm, vias 0 -> 1
- net DIG_2: track 0.00 -> 15.6 mm, vias 0 -> 1
- net SEG_P: track 0.00 -> 13.5 mm, vias 0 -> 1
- net SEG_G: track 2.80 -> 15.1 mm, vias 0 -> 1
- net SEG_A/A2: track 30.2 -> 41.3 mm, vias 1 -> 2
- net VUSB: track 0.00 -> 9.30 mm
- net SEG_B/A1/COL_A: track 21.0 -> 29.5 mm, vias 0 -> 1
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Other:
- board text added: "7 Segement"
- board text added: "Feather Wing"
