File: hardware/tick-pi-mk-1.1.brd (EAGLE design)
At the start: 66 x 38.1 mm, 15 parts, among them Q1 N6040

Commit message: more pi boards
Parts:
- C1: value 10uF -> 4u7
- C2: value 1uF -> 1u; device a_parts:C0805-TIGHTER -> a_parts:C0603-TIGHTER
- JP6: value (none) -> M081X08; device a_parts:1X07 -> a_parts:1X08
- JP7: value M04X2PTH -> M02PTH-CENTERED; device a_parts:2X4_PTH -> a_parts:1X02-CENTER
- Q1: value N6040 -> IRF7341
- moved C1 44.9 mm to (12.7, 34.9), flipped to the top
- moved C2 24.4 mm to (33.0, 15.9), flipped to the top
- moved JP5 8.13 mm to (47.0, 35.6), turned to 180 degrees
- moved JP1 6.48 mm to (33.0, 30.5), flipped to the top
- moved R2 5.08 mm to (26.7, 17.8)
- moved R4 5.08 mm to (39.4, 17.8)
- moved Q1 5.08 mm to (33.0, 20.3)
- moved JP7 4.49 mm to (61.6, 17.1), flipped to the bottom, turned to 90 degrees
- moved R1 4.45 mm to (26.7, 22.2)
- moved R3 4.45 mm to (39.4, 22.2), turned to 270 degrees
- moved JP6 2.29 mm to (24.1, 9.53), flipped to the bottom, turned to 180 degrees
Connections:
- new net GPIO21: JP1.40, JP7.2
- new net RX: JP1.10, JP6.8
- net 3.3V: no longer JP5.2, JP7.1
- net 5V: now also JP5.2; no longer JP7.2, JP7.4
- net GND: now also JP7.1; no longer JP7.6
- net GPIO4: no longer JP7.7
- net SCL_3V: no longer JP5.4, JP7.5
- net SCL_5V: now also JP5.4
- net SDA_3V: no longer JP5.3, JP7.3
- net SDA_5V: now also JP5.3
- net TX: no longer JP7.8
Routing:
- net SCL_5V: track 96.5 -> 131.6 mm, vias 2 -> 4
- net RX: track 0.00 -> 34.7 mm, vias 0 -> 1
- net SDA_3V: track 75.9 -> 43.5 mm, vias 3 -> 1
- net SCL_3V: track 70.8 -> 38.7 mm, vias 3 -> 1
- net 3.3V: track 97.5 -> 69.5 mm, vias 2 -> 0
- net SDA_5V: track 111.7 -> 130.2 mm
- net GPIO21: track 0.00 -> 15.2 mm
- net GPIO4: track 44.6 -> 31.1 mm, vias 1 -> 0
- net TX: track 42.6 -> 34.7 mm, vias 0 -> 1
- net 5V: track 164.6 -> 158.3 mm, vias 2 -> 0
- net GND: track 0.00 -> 5.77 mm, vias 0 -> 1
Other:
- board text added: "21"
- board text added: "4"
- board text added: "DISPLAY SIDE"
- board text added: "RASPBERRY PI SIDE"
- board text added: "RX"
- board text removed: "GP4"
