File: hardware/tick-pi-mk-1.1.sch (EAGLE design)
At the start: 15 parts, among them Q1 N6040

Commit message: more pi boards
Parts:
- C1: value 10uF -> 4u7
- C2: value 1uF -> 1u; device a_parts:CAPACITOR-CERAMICC0805-TIGHTER -> a_parts:CAPACITOR-CERAMICC0603-TIGHTER
- FRAME1: VERSION v1.0 -> v1.1
- JP6: value (none) -> M081X08; device a_parts:M07 -> a_parts:M081X08
- JP7: value M04X2PTH -> M02PTH-CENTERED; device a_parts:M04X2PTH -> a_parts:M02PTH-CENTERED
- Q1: value N6040 -> IRF7341
Connections:
- new net GPIO21: JP1.GP21, JP7.2
- new net RX: JP1.RXI, JP6.8
- net 3.3V: no longer JP5.2, JP7.1
- net 5V: now also JP5.2; no longer JP7.2, JP7.4
- net GND: now also JP7.1; no longer JP7.6
- net GPIO4: no longer JP7.7
- net SCL_3V: no longer JP5.4, JP7.5
- net SCL_5V: now also JP5.4
- net SDA_3V: no longer JP5.3, JP7.3
- net SDA_5V: now also JP5.3
- net TX: no longer JP7.8
